Commit message: urdf end

File: urdf/urdf.urdf (robot description, URDF)
Before this commit: robot robot, 2 links, 1 joints
Links:
- added link loadcell; visual mesh filename=package://PID/meshs/loadcell.stl scale=0.1 0.1 0.1
- added link loadcell_plate; visual mesh filename=package://PID/meshs/loadcell_plate.stl scale=0.1 0.1 0.1
- added link loadcell_pressure; visual mesh filename=package://PID/meshs/loadcell_pressure.stl scale=0.1 0.1 0.1
- added link servo_arm; visual mesh filename=package://PID/meshs/servo_arm.stl scale=0.1 0.1 0.1
- added link servo_support; visual mesh filename=package://PID/meshs/servo_support.stl scale=0.1 0.1 0.1
Joints:
- removed joint j1
- added joint base_to_dc: type revolute, parent base_link, child dc_roller, origin xyz=25 -8 3 rpy=0 0 0, axis 0 1 0, limit lower=-3.14 upper=3.14 effort=20 velocity=5
- added joint j2: type fixed, parent base_link, child loadcell_plate, origin xyz=5 -3 0 rpy=0 0 0, axis 0 0 0
- added joint j3: type fixed, parent loadcell_plate, child loadcell, origin xyz=0 1 3 rpy=0 0 0, axis 0 0 0
- added joint j4: type fixed, parent loadcell_plate, child loadcell_pressure, origin xyz=0 2.6 4 rpy=0 0 0, axis 0 0 0
- added joint j5: type fixed, parent base_link, child servo_support, origin xyz=15 -4 0 rpy=0 0 0, axis 0 0 0
- added joint servo_to_arm: type revolute, parent servo_support, child servo_arm, origin xyz=0 3 5 rpy=0 0 0, axis 0 1 0, limit lower=-0.8 upper=2.35 effort=20 velocity=5

Commit message: joint state publusher and launch files

File: urdf/urdf.urdf (robot description, URDF)
Before this commit: robot robot, 7 links, 6 joints
Joints:
- joint base_to_dc: limit lower=-3.14 upper=3.14 effort=20 velocity=5 -> (none); type revolute -> fixed
